Commit message: limits in rad (as in unitree repo)

File: urdfs/const.xacro (robot description, xacro)
@@ -43,6 +43,18 @@
     <xacro:property name="kfe_motor_offset_z" value="0.0"/>
     <!-- joint limits -->
-    <xacro:property name="damping" value="0.00"/>
+    <!-- xacro:property name="damping" value="0.00"/>
     <xacro:property name="friction" value="0.0"/>
+    <xacro:property name="haa_max" value="${20*PI}"/>
+    <xacro:property name="haa_min" value="${-20*PI}"/>
+    <xacro:property name="haa_velocity_max" value="3000"/>
+    <xacro:property name="haa_torque_max" value="2370"/>
+    <xacro:property name="hfe_max" value="${20*PI}"/>
+    <xacro:property name="hfe_min" value="${-20*PI}"/>
+    <xacro:property name="hfe_velocity_max" value="3000"/>
+    <xacro:property name="hfe_torque_max" value="2370"/>
+    <xacro:property name="kfe_max" value="${20*PI}"/>
+    <xacro:property name="kfe_min" value="${-20*PI}"/>
+    <xacro:property name="kfe_velocity_max" value="3000"/>
+    <xacro:property name="kfe_torque_max" value="2370"/ -->
     <xacro:property name="haa_max" value="0.863"/>
     <xacro:property name="haa_min" value="-0.863"/>
@@ -56,5 +68,5 @@
     <xacro:property name="kfe_min" value="-2.818"/>
     <xacro:property name="kfe_velocity_max" value="20.06"/>
-    <xacro:property name="kfe_torque_max" value="35.55"/>
+    <xacro:property name="kfe_torque_max" value="35.55">
     <!-- dynamics inertial value        total 12.84kg -->
     <!-- trunk -->

File: urdfs/leg.xacro (robot description, xacro)
@@ -12,8 +12,10 @@
             <dynamics damping="${damping}" friction="${friction}"/>
             <xacro:if value="${(mirror_dae == True)}">
-                <limit effort="${haa_torque_max}" velocity="${haa_velocity_max}" lower="${haa_min}" upper="${haa_max}"/>
+                <!-- limit effort="${haa_torque_max}" velocity="${haa_velocity_max}" lower="${haa_min*PI/180.0}" upper="${haa_max*PI/180.0}"/ -->
+                <limit effort="${haa_torque_max}" velocity="${haa_velocity_max}" lower="${haa_min}" upper="${haa_max}" />
             </xacro:if>
             <xacro:if value="${(mirror_dae == False)}">
-                <limit effort="${haa_torque_max}" velocity="${haa_velocity_max}" lower="${-haa_max}" upper="${-haa_min}"/>
+                <!-- limit effort="${haa_torque_max}" velocity="${haa_velocity_max}" lower="${-haa_max*PI/180.0}" upper="${-haa_min*PI/180.0}"/ -->
+                <limit effort="${haa_torque_max}" velocity="${haa_velocity_max}" lower="${-haa_max}" upper="${-haa_min}" />
             </xacro:if>
         </joint>
@@ -112,4 +114,5 @@
             <axis xyz="0 1 0"/>
             <dynamics damping="${damping}" friction="${friction}"/>
+            <!--limit effort="${hfe_torque_max}" velocity="${hfe_velocity_max}" lower="${hfe_min*PI/180.0}" upper="${hfe_max*PI/180.0}"/ -->
             <limit effort="${hfe_torque_max}" velocity="${hfe_velocity_max}" lower="${hfe_min}" upper="${hfe_max}"/>
         </joint>
@@ -188,4 +191,5 @@
             <axis xyz="0 1 0"/>
             <dynamics damping="${damping}" friction="${friction}"/>
+            <!-- limit effort="${kfe_torque_max}" velocity="${kfe_velocity_max}" lower="${kfe_min*PI/180.0}" upper="${kfe_max*PI/180.0}"/ -->
             <limit effort="${kfe_torque_max}" velocity="${kfe_velocity_max}" lower="${kfe_min}" upper="${kfe_max}"/>
         </joint>
